File: ax5243/ax5243_feather/ax5243_feather.brd (EAGLE design)
At the start: 22.9 x 50.8 mm, 21 parts

Commit message: catching up commits, can't remember whats new in this one.
Parts:
- L1, L2, L3, L4, L5, L6, L7: device rcl:L2012C -> kj4qlp:C0805K
- X1: value (none) -> RF
- moved L5 1.98 mm to (6.60, 42.7), turned to 270 degrees
- moved C5 1.70 mm to (6.60, 38.9), turned to 270 degrees
- moved L6 1.55 mm to (13.7, 41.7)
- moved C8 1.27 mm to (14.5, 44.5)
- moved L7 1.27 mm to (12.7, 44.5)
- moved L3 1.05 mm to (13.7, 39.9)
- moved C1 1.02 mm to (15.2, 34.3)
- moved C7 1.02 mm to (16.3, 42.4)
- moved Q1 0.92 mm to (17.0, 29.0)
- moved L1 0.80 mm to (15.2, 36.1)
- moved C6 0.80 mm to (9.40, 41.7)
- moved L4 0.80 mm to (9.40, 39.9)
- moved C9 0.76 mm to (9.40, 43.4)
- moved L2 0.57 mm to (7.37, 36.1)
- moved C10 0.57 mm to (9.14, 45.2)
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Routing:
- net GND: track 29.7 -> 65.2 mm, vias 16 -> 50
- net N$1: track 0.00 -> 2.49 mm
- net N$8: track 7.16 -> 8.93 mm
- net N$9: track 7.19 -> 8.19 mm
- net N$11: track 5.88 -> 6.87 mm
- net N$3: track 2.33 -> 3.28 mm
- net N$4: track 2.51 -> 3.40 mm
- net N$6: track 1.55 -> 2.30 mm
- net ANTP: track 5.50 -> 6.17 mm
- net N$10: track 5.24 -> 4.66 mm
- net N$7: track 4.89 -> 5.40 mm
- added copper zone on layer 1, net GND
Other:
- board text added: "MISO"
- board text added: "MOSI"
