File: rfm69/rfm69_32u4/rev-/rfm69_32u4.sch (EAGLE design)
At the start: 36 parts, among them K1 G5LE, SW1 SPST_TACT-KMR2, U1 433MHz, X2 USB-A, Y1 8MHz

Commit message: minor changes
Parts:
- added LED3: FIX, adafruit:LEDCHIPLED_0805
- added R10: 10k, adafruit:R-US_R0805
- LED2: value (none) -> RELAY
- U$5: value (none) -> CH291-1220LF; device adafruit:CR1220SMT -> battery:CH291-1220LF
- X2: value USB-A -> USB_B_PTH; device adafruit:USB-A -> SparkFun-Connectors:USB_B_PTH
Connections:
- net A4_RF_RST renamed A4
- removed net 10: U$1.PB6(OC1B/OC4B/ADC13)
- removed net 11: U$1.PB7(OC0A/OC1C/RTS)
- removed net 13: U$1.PC7(ICP3/CLK0/OC4A)
- removed net 5: U$1.PC6(OC3A/!OC4A)
- removed net 6: U$1.PD7(OC4D/ADC10/T0)
- removed net 8: LED1.A, U$1.PB4(ADC11)
- removed net A0: U$1.PF7(ADC7(TDI)
- removed net GPS_PPS: U$1.PD0(INT0/OC0B/SCL)
- removed net GPS_RST: U2.NRESET
- removed net GPS_RXD: U2.RX
- removed net GPS_TXD: U2.TX
- removed net PPS: U2.1PPS
- removed net RF_RST: R6.2, U1.RESET
- removed net TXLED: U$1.PD5(XCK/CTS)
- removed net X_RF_DIO1: U1.DIO1
- removed net X_RF_DIO2: U1.DIO2
- removed net X_RF_DIO3: U1.DIO3
- removed net X_RF_DIO4: U1.DIO4
- removed net X_RF_DIO5: U1.DIO5
- new net 10_RF_DIO5: U$1.PB6(OC1B/OC4B/ADC13), U1.DIO5
- new net 11_LED: LED1.A, U$1.PB7(OC0A/OC1C/RTS)
- new net 13_RF_DIO4: U$1.PC7(ICP3/CLK0/OC4A), U1.DIO4
- new net 22_RF_RST: R6.2, U$1.PD5(XCK/CTS), U1.RESET
- new net 3_GPS_PPS: U$1.PD0(INT0/OC0B/SCL), U2.1PPS
- new net 5_RF_DIO3: U$1.PC6(OC3A/!OC4A), U1.DIO3
- new net 6_RF_DIO1: U$1.PD7(OC4D/ADC10/T0), U1.DIO1
- new net 8_RF_DIO2: U$1.PB4(ADC11), U1.DIO2
- new net A0_GPS_RST: U$1.PF7(ADC7(TDI), U2.NRESET
- new net N$5: LED3.C, R10.2
- net 0_GPS_TXD: now also U2.TX
- net 1_GPS_RXD: now also U2.RX
- net 3D-FIX: now also LED3.A
- net GND: now also R10.1, U$5.-
- net VBACKUP: now also U$5.+
Other:
- moved on the sheet: GPS_ANT
